Commit message: Lock joints

File: environments/3d_models/robots/shadow_hand.urdf (robot description, URDF)
Before this commit: robot shadowhand, 35 links, 34 joints
Joints:
- joint FFJ4: limit lower=0.43633231299858238 upper=-0.43633231299858238 effort=100 velocity=5.0 -> lower=-0.43633231299858238 upper=0.0 effort=100 velocity=5.0
- joint LFJ4: limit lower=0.43633231299858238 upper=-0.43633231299858238 effort=100 velocity=5.0 -> lower=-0.43633231299858238 upper=0.0 effort=100 velocity=5.0
- joint MFJ4: limit lower=0.43633231299858238 upper=-0.43633231299858238 effort=100 velocity=5.0 -> lower=-0.43633231299858238 upper=0 effort=100 velocity=5.0
- joint RFJ4: limit lower=0.43633231299858238 upper=-0.43633231299858238 effort=100 velocity=5.0 -> lower=-0.43633231299858238 upper=0.0 effort=100 velocity=5.0
